File: KiCad/DuoPad.kicad_pcb (KiCad board)
At the start: 2 copper layers, 113.7 x 120.7 mm, 7 parts, among them SW1 SW_Push, SW2 RotaryEncoder_Switch, SW3 SW_Push, SW4 SW_Push, SW5 SW_Push, SW6 SW_Push, U1 nice_nano

Commit message: Add files via upload
Parts:
- moved SW2 0.84 mm to (154.4, 54.6)
Routing:
- net GND: track 260.7 -> 256.4 mm
- net AIN7/P0.31: track 58.1 -> 56.4 mm
Changed lines of the file:
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@@
 	(footprint "Rotary_Encoder:RotaryEncoder_Alps_EC11E-Switch_Vertical_H20mm_MountingHoles"
 		(layer "F.Cu")
-		(at 154.425 55.4875)
+		(at 154.425 54.65)
 		(descr "Alps rotary encoder, EC11E... with switch, vertical shaft, https://www.lcsc.com/datasheet/lcsc_datasheet_2410010003_ALPSALPINE-EC11E09444A8_C1322538.pdf")
 		(tags "rotary encoder")
@@
 		(layer "F.SilkS")
 	)
+	(gr_line
+		(start 155.42497 50.15)
+		(end 168.42485 50.15)
+		(stroke
+			(width 0.2)
+			(type default)
+		)
+		(layer "F.SilkS")
+	)
 	(gr_arc
 		(start 143.5189 142.73125)
@@
 	)
 	(gr_line
+		(start 168.925 50.657171)
+		(end 168.925 63.65)
+		(stroke
+			(width 0.2)
+			(type default)
+		)
+		(layer "F.SilkS")
+	)
+	(gr_line
 		(start 143.5189 142.73125)
 		(end 156.51875 142.73125)
@@
 	)
 	(gr_line
+		(start 155.42515 64.15)
+		(end 168.425 64.15)
+		(stroke
+			(width 0.2)
+			(type default)
+		)
+		(layer "F.SilkS")
+	)
+	(gr_arc
+		(start 168.42485 50.15)
+		(mid 168.778521 50.296464)
+		(end 168.925 50.657171)
+		(stroke
+			(width 0.2)
+			(type default)
+		)
+		(layer "F.SilkS")
+	)
+	(gr_line
+		(start 154.925 50.64997)
+		(end 154.925 63.6569)
+		(stroke
+			(width 0.2)
+			(type default)
+		)
+		(layer "F.SilkS")
+	)
+	(gr_line
 		(start 157.01875 129.238421)
 		(end 157.01875 142.23125)
@@
 		(start 166.6875 145.25625)
 		(end 166.6875 126.20625)
+		(stroke
+			(width 0.2)
+			(type default)
+		)
+		(layer "F.SilkS")
+	)
+	(gr_arc
+		(start 168.925 63.65)
+		(mid 168.778556 64.003571)
+		(end 168.425 64.15)
+		(stroke
+			(width 0.2)
+			(type default)
+		)
+		(layer "F.SilkS")
+	)
+	(gr_arc
+		(start 155.42515 64.15)
+		(mid 155.071479 64.003536)
+		(end 154.925 63.6569)
 		(stroke
 			(width 0.2)
@@
 		(mid 143.165194 128.877679)
 		(end 143.51872 128.73125)
+		(stroke
+			(width 0.2)
+			(type default)
+		)
+		(layer "F.SilkS")
+	)
+	(gr_arc
+		(start 154.925 50.64997)
+		(mid 155.071444 50.296429)
+		(end 155.42497 50.15)
 		(stroke
 			(width 0.2)
@@
 	(segment
 		(start 171.45 50.00625)
-		(end 171.45 54.76875)
+		(end 171.45 52.3875)
+		(width 0.2)
+		(layer "F.Cu")
+		(net 2)
+	)
+	(segment
+		(start 150.7375 57.15)
+		(end 154.425 57.15)
 		(width 0.2)
 		(layer "F.Cu")
@@
 	)
 	(segment
-		(start 145.25625 57.15)
-		(end 146.09375 57.9875)
-		(width 0.2)
-		(layer "F.Cu")
-		(net 2)
-	)
-	(segment
 		(start 121.6025 97.63125)
 		(end 126.0475 102.07625)
@@
 	)
 	(segment
-		(start 146.09375 57.9875)
-		(end 154.425 57.9875)
-		(width 0.2)
-		(layer "F.Cu")
-		(net 2)
-	)
-	(segment
 		(start 168.709375 47.265625)
 		(end 171.45 50.00625)
@@
 	(segment
 		(start 140.853125 47.265625)
-		(end 145.25625 51.66875)
+		(end 150.7375 57.15)
 		(width 0.2)
 		(layer "F.Cu")
@@
 	)
 	(segment
-		(start 145.25625 51.66875)
-		(end 145.25625 57.15)
-		(width 0.2)
-		(layer "F.Cu")
-		(net 2)
-	)
-	(segment
 		(start 142.875 97.63125)
 		(end 145.0975 99.85375)
@@
 	)
 	(segment
+		(start 168.925 54.65)
+		(end 169.1875 54.65)
+		(width 0.2)
+		(layer "F.Cu")
+		(net 2)
+	)
+	(segment
 		(start 152.4 111.60125)
 		(end 152.4 97.63125)
@@
 	)
 	(segment
+		(start 169.1875 54.65)
+		(end 171.45 52.3875)
+		(width 0.2)
+		(layer "F.Cu")
+		(net 2)
+	)
+	(segment
 		(start 115.8875 40.08)
 		(end 115.8875 42.62)
@@
 	)
 	(segment
-		(start 171.45 54.76875)
-		(end 169.64375 54.76875)
-		(width 0.2)
-		(layer "F.Cu")
-		(net 2)
-	)
-	(segment
 		(start 111.91875 95.25)
 		(end 114.3 97.63125)
@@
 	)
 	(segment
+		(start 142.875 59.53125)
+		(end 142.99375 59.65)
+		(width 0.2)
+		(layer "F.Cu")
+		(net 3)
+	)
+	(segment
 		(start 140.49375 57.15)
-		(end 143.83125 60.4875)
+		(end 142.875 59.53125)
 		(width 0.2)
 		(layer "F.Cu")
@@
 	)
 	(segment
-		(start 143.83125 60.4875)
-		(end 154.425 60.4875)
+		(start 142.99375 59.65)
+		(end 154.425 59.65)
 		(width 0.2)
 		(layer "F.Cu")
@@
 	)
 	(segment
+		(start 171.45 57.15)
+		(end 173.83125 54.76875)
+		(width 0.2)
+		(layer "B.Cu")
+		(net 4)
+	)
+	(segment
 		(start 168.985 45.16)
 		(end 173.83125 50.00625)
@@
 	)
 	(segment
-		(start 170.49375 60.4875)
-		(end 168.925 60.4875)
+		(start 171.425 57.15)
+		(end 171.45 57.15)
 		(width 0.2)
 		(layer "B.Cu")
@@
 	)
 	(segment
-		(start 173.83125 57.15)
-		(end 170.49375 60.4875)
+		(start 173.83125 50.00625)
+		(end 173.83125 54.76875)
 		(width 0.2)
 		(layer "B.Cu")
@@
 	)
 	(segment
-		(start 173.83125 50.00625)
-		(end 173.83125 57.15)
+		(start 171.425 57.15)
+		(end 168.925 59.65)
 		(width 0.2)
 		(layer "B.Cu")
@@
 	)
 	(segment
+		(start 147.51875 54.65)
+		(end 154.425 54.65)
+		(width 0.2)
+		(layer "B.Cu")
+		(net 5)
+	)
+	(segment
 		(start 143.10875 50.24)
-		(end 148.35625 55.4875)
+		(end 131.1275 50.24)
 		(width 0.2)
 		(layer "B.Cu")
@@
 	)
 	(segment
-		(start 131.1275 50.24)
+		(start 146.425375 53.556625)
 		(end 143.10875 50.24)
 		(width 0.2)
@@
 	)
 	(segment
-		(start 148.35625 55.4875)
-		(end 154.425 55.4875)
+		(start 146.425375 53.556625)
+		(end 147.51875 54.65)
 		(width 0.2)
 		(layer "B.Cu")
@@
 	)
 	(group ""
+		(members "02e8834f-20d3-4454-a144-8985b5072e32" "0c4a8c21-7c00-4225-8243-f6a66451e4b5"
+			"84491c31-1411-4628-a353-17dec0745bc9" "90b88eed-d60c-4837-9288-dac342dc9743"
+			"a6157855-14b8-4f87-8835-a56dbb7811cc" "ad51f69f-cd5d-4dda-b7a7-7b4e5082917f"
+			"bb4bb435-fb40-42cc-a28e-cea06ee9fe46" "d457e0b7-ee3a-4935-bcdd-6c8ec71c7506"
+			"d47bb665-5d6b-4911-9b5d-56ae5a3b27d7" "ea904161-dc95-4a7b-a656-95b0b93a6714"
+		)
+	)
+	(group ""
